Commit message: modified gripper collision

File: mycobot_280/mycobot_280m5_gazebo_gripper/config/mycobot_280m5_with_gripper_lll.urdf (robot description, URDF)
Before this commit: robot firefighter, 15 links, 14 joints
Links:
- link gripper_left1: geometry collision box size=0.011 0.02 0.02; visual mesh filename=package://mycobot_description/urdf/mycobot_280_m5/gripper_l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
- link gripper_right1: geometry collision box size=0.011 0.02 0.02; visual mesh filename=package://mycobot_description/urdf/mycobot_280_m5/gripper_r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
